Commit message: Modify the upper body URDF

File: urdf/dobot_atom.urdf (robot description, URDF)
Before this commit: robot atom, 20 links, 19 joints
Links:
- removed link pelvis
Joints:
- removed joint base_joint
- joint torso_joint: parent pelvis -> base_link

File: xacro/component.xacro (robot description, xacro)
@@ -9,5 +9,5 @@
 	<xacro:if value="${'$(arg type)' == 'upper_body'}">
 		<xacro:include filename="$(find dobot_atom_description)/xacro/upper_body.xacro"/>
-		<xacro:AtomUpperBody parent_link="base_link"/>
+		<xacro:AtomUpperBody parent_link="base_link" type="$(arg type)"/>
 	</xacro:if>
 	<xacro:if value="${'$(arg type)' == 'left_arm'}">

File: xacro/full_upper_body.xacro (robot description, xacro)
@@ -5,16 +5,4 @@
 <robot name="atom" xmlns:xacro="http://www.ros.org/wiki/xacro">
 	<xacro:property name="type" value="upper"/>
-	<link name="pelvis">
-		<inertial>
-			<origin xyz="0.0006 0.0000 -0.0998"/>
-			<mass value="6.5370"/>
-			<inertia ixx="0.0344" ixy="0.0000" ixz="0.0001" iyy="0.0292" iyz="0.0000" izz="0.0214"/>
-		</inertial>
-		<visual>
-			<geometry>
-				<mesh filename="file://$(find dobot_atom_description)/meshes/body/pelvis.obj"/>
-			</geometry>
-		</visual>
-	</link>
 	<!-- Without Left Leg -->
 	<!-- xacro:include filename="$(find dobot_atom_description)/xacro/leg.xacro"/>
@@ -24,5 +12,5 @@
 	<!-- Upper Body (Torso, Head, IMU) -->
 	<xacro:include filename="$(find dobot_atom_description)/xacro/upper_body.xacro"/>
-	<xacro:AtomUpperBody parent_link="pelvis" type="upper"/>
+	<xacro:AtomUpperBody parent_link="base_link" type="upper"/>
 	<!-- Left Arm -->
 	<xacro:include filename="$(find dobot_atom_description)/xacro/arm.xacro"/>

File: xacro/robot.xacro (robot description, xacro)
@@ -5,10 +5,13 @@
 <robot name="atom" xmlns:xacro="http://www.ros.org/wiki/xacro">
 	<link name="base_link"/>
-	<joint name="base_joint" type="fixed">
-		<parent link="base_link"/>
-		<child link="pelvis"/>
-	</joint>
 	<!-- 切换模式参数 -->
 	<xacro:arg name="type" default="full" />
+    <!-- 当为 full 模式时，创建 base_link -> pelvis 连接 -->
+    <xacro:if value="${'$(arg type)' == 'full'}">
+    	<joint name="base_joint" type="fixed">
+    		<parent link="base_link"/>
+    		<child link="pelvis"/>
+    	</joint>
+    </xacro:if>
 	<!-- 全身模式 -->
     <xacro:if value="${'$(arg type)' == 'full'}">

Commit message: Update self collision

File: urdf/dobot_atom.urdf (robot description, URDF)
Before this commit: robot atom, 19 links, 18 joints
Links:
- link left_elbow_pitch_link: geometry collision cylinder length=0.11 radius=0.04; visual mesh filename=file:///home/ly/ros2_ws/install/dobot_atom_description/shar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
- link left_elbow_roll_link: geometry collision cylinder length=0.15 radius=0.045; visual mesh filename=file:///home/ly/ros2_ws/install/dobot_atom_description/shar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
- link left_shoulder_roll_link: geometry visual mesh filename=file:///home/ly/ros2_ws/install/dobot_atom_description/shar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 scale=1 1 1
- link left_shoulder_yaw_link: geometry collision cylinder length=0.20 radius=0.04; visual mesh filename=file:///home/ly/ros2_ws/install/dobot_atom_description/shar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
- link left_wrist_pitch_link: geometry collision cylinder length=0.09 radius=0.035; visual mesh filename=file:///home/ly/ros2_ws/install/dobot_atom_description/shar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 scale=1 1 1
- link left_wrist_yaw_link: geometry collision cylinder length=0.09 radius=0.035; visual mesh filename=file:///home/ly/ros2_ws/install/dobot_atom_description/shar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 scale=1 1 1
- link right_elbow_pitch_link: geometry collision cylinder length=0.11 radius=0.04; visual mesh filename=file:///home/ly/ros2_ws/install/dobot_atom_description/shar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
- link right_elbow_roll_link: geometry collision cylinder length=0.15 radius=0.045; visual mesh filename=file:///home/ly/ros2_ws/install/dobot_atom_description/shar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
- link right_shoulder_roll_link: geometry visual mesh filename=file:///home/ly/ros2_ws/install/dobot_atom_description/shar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 scale=1 -1 1
- link right_shoulder_yaw_link: geometry collision cylinder length=0.20 radius=0.04; visual mesh filename=file:///home/ly/ros2_ws/install/dobot_atom_description/shar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
- link right_wrist_pitch_link: geometry collision cylinder length=0.09 radius=0.035; visual mesh filename=file:///home/ly/ros2_ws/install/dobot_atom_description/shar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 scale=1 -1 1
- link right_wrist_yaw_link: geometry collision cylinder length=0.09 radius=0.035; visual mesh filename=file:///home/ly/ros2_ws/install/dobot_atom_description/shar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 scale=1 -1 1

File: xacro/arm.xacro (robot description, xacro)
@@ -35,10 +35,4 @@
 				</geometry>
 			</visual>
-			<collision>
-				<origin xyz="0 0 -0.1"/>
-				<geometry>
-					<box size="0.06 0.06 0.24"/>
-				</geometry>
-			</collision>
 		</link>
 		<joint name="${prefix}shoulder_roll_joint" type="revolute">
@@ -62,4 +56,10 @@
 				</geometry>
 			</visual>
+			<collision>
+				<origin xyz="0 0 0"/>
+				<geometry>
+					<cylinder radius="0.04" length="0.20"/>
+				</geometry>
+			</collision>
 		</link>
 		<joint name="${prefix}shoulder_yaw_joint" type="revolute">
@@ -84,7 +84,7 @@
 			</visual>
 			<collision>
-				<origin xyz="0.16 0 0"/>
+				<origin rpy="1.57079632679 0 0"/>
 				<geometry>
-					<box size="0.30 0.06 0.06"/>
+					<cylinder radius="0.04" length="0.11"/>
 				</geometry>
 			</collision>
@@ -109,4 +109,12 @@
 				</geometry>
 			</visual>
+			<collision>
+                <origin
+				    xyz="-0.04 0 0"
+				    rpy="0 1.57079632679 0"/>
+                <geometry>
+                    <cylinder radius="0.045" length="0.15"/>
+                </geometry>
+            </collision>
 		</link>
 		<joint name="${prefix}elbow_roll_joint" type="revolute">
@@ -129,4 +137,10 @@
 				</geometry>
 			</visual>
+			<collision>
+				<origin rpy="1.57079632679 0 0"/>
+				<geometry>
+					<cylinder radius="0.035" length="0.09"/>
+				</geometry>
+			</collision>
 		</link>
 		<joint name="${prefix}wrist_pitch_joint" type="revolute">
@@ -149,4 +163,10 @@
 				</geometry>
 			</visual>
+			<collision>
+                <origin rpy="0 0 0"/>
+                <geometry>
+                    <cylinder radius="0.035" length="0.09"/>
+                </geometry>
+            </collision>
 		</link>
 		<joint name="${prefix}wrist_yaw_joint" type="revolute">

File: xacro/ros2_control/robot.xacro (robot description, xacro)
@@ -8,7 +8,5 @@
 	<xacro:arg name="ros2_control_hardware_type" default="mock_components"/>
   <!-- include the main robot definition (this file defines links/joints/macros) -->
-  <xacro:include filename="$(find dobot_atom_description)/xacro/robot.xacro">
-    <xacro:arg name="type" value="$(arg type)"/>
-  </xacro:include>
+  <xacro:include filename="$(find dobot_atom_description)/xacro/robot.xacro"/>
   <!-- Import modular interface components -->
   <xacro:include filename="$(find dobot_atom_description)/xacro/ros2_control/atom_head_interfaces.xacro"/>
